Commit message: 成功添加/home/dw/workspace/opendog_ros2/src/ocs2_ros2/advance examples/ocs2_perceptive_anymal/ocs2_anymal_loopshaping_mpc/launch/togo_prototype.launch.py

File: src/ToGo.Prototype/urdf/ToGo.Prototype.urdf (robot description, URDF)
Before this commit: robot Xtellar.Robotics/ToGo.Prototype, 19 links, 18 joints
Links:
- added link Lfl4_wheel_contact
- added link Lfr4_wheel_contact
- added link Lrl4_wheel_contact
- added link Lrr4_wheel_contact
Joints:
- added joint Jfl4_wheel_contact: type fixed, parent Lfl4_wheel, child Lfl4_wheel_contact, origin xyz=0.000000000e+00 -7.898243040e-02 4.314829848e-02 rpy=0.000000000e+00 0.000000000e+00 0.000000000e+00
- added joint Jfr4_wheel_contact: type fixed, parent Lfr4_wheel, child Lfr4_wheel_contact, origin xyz=0.000000000e+00 -7.898243040e-02 4.314829848e-02 rpy=0.000000000e+00 0.000000000e+00 0.000000000e+00
- added joint Jrl4_wheel_contact: type fixed, parent Lrl4_wheel, child Lrl4_wheel_contact, origin xyz=0.000000000e+00 -7.898243040e-02 4.314829848e-02 rpy=0.000000000e+00 0.000000000e+00 0.000000000e+00
- added joint Jrr4_wheel_contact: type fixed, parent Lrr4_wheel, child Lrr4_wheel_contact, origin xyz=0.000000000e+00 -7.898243040e-02 4.314829848e-02 rpy=0.000000000e+00 0.000000000e+00 0.000000000e+00
- joint J1_waist: axis 0.000000000e+00 -1.000000000e+00 0.000000000e+00 -> (none); limit lower=-0.026179938779914945 upper=0.026179938779914945 effort=97.0 velocity=6.283185307179586 -> (none); type revolute -> fixed
- joint Jfl4_wheel: axis 1.000000000e+00 0.000000000e+00 0.000000000e+00 -> (none); limit lower=0.0 upper=0.0 effort=40.0 velocity=33.510321638291124 -> (none); type continuous -> fixed
- joint Jfr4_wheel: axis -1.000000000e+00 0.000000000e+00 0.000000000e+00 -> (none); limit lower=0.0 upper=0.0 effort=40.0 velocity=33.510321638291124 -> (none); type continuous -> fixed
- joint Jrl4_wheel: axis 1.000000000e+00 0.000000000e+00 0.000000000e+00 -> (none); limit lower=0.0 upper=0.0 effort=40.0 velocity=33.510321638291124 -> (none); type continuous -> fixed
- joint Jrr4_wheel: axis -1.000000000e+00 0.000000000e+00 0.000000000e+00 -> (none); limit lower=0.0 upper=0.0 effort=40.0 velocity=33.510321638291124 -> (none); type continuous -> fixed

File: src/ToGo.Prototype/urdf/ToGo.Prototype_abs.urdf (robot description, URDF)
Before this commit: robot Xtellar.Robotics/ToGo.Prototype, 19 links, 18 joints
Links:
- added link Lfl4_wheel_contact
- added link Lfr4_wheel_contact
- added link Lrl4_wheel_contact
- added link Lrr4_wheel_contact
Joints:
- added joint Jfl4_wheel_contact: type fixed, parent Lfl4_wheel, child Lfl4_wheel_contact, origin xyz=0.000000000e+00 -7.898243040e-02 4.314829848e-02 rpy=0.000000000e+00 0.000000000e+00 0.000000000e+00
- added joint Jfr4_wheel_contact: type fixed, parent Lfr4_wheel, child Lfr4_wheel_contact, origin xyz=0.000000000e+00 -7.898243040e-02 4.314829848e-02 rpy=0.000000000e+00 0.000000000e+00 0.000000000e+00
- added joint Jrl4_wheel_contact: type fixed, parent Lrl4_wheel, child Lrl4_wheel_contact, origin xyz=0.000000000e+00 -7.898243040e-02 4.314829848e-02 rpy=0.000000000e+00 0.000000000e+00 0.000000000e+00
- added joint Jrr4_wheel_contact: type fixed, parent Lrr4_wheel, child Lrr4_wheel_contact, origin xyz=0.000000000e+00 -7.898243040e-02 4.314829848e-02 rpy=0.000000000e+00 0.000000000e+00 0.000000000e+00
- joint J1_waist: axis 0.000000000e+00 -1.000000000e+00 0.000000000e+00 -> (none); limit lower=-0.026179938779914945 upper=0.026179938779914945 effort=97.0 velocity=6.283185307179586 -> (none); type revolute -> fixed
- joint Jfl4_wheel: axis 1.000000000e+00 0.000000000e+00 0.000000000e+00 -> (none); limit lower=0.0 upper=0.0 effort=40.0 velocity=33.510321638291124 -> (none); type continuous -> fixed
- joint Jfr4_wheel: axis -1.000000000e+00 0.000000000e+00 0.000000000e+00 -> (none); limit lower=0.0 upper=0.0 effort=40.0 velocity=33.510321638291124 -> (none); type continuous -> fixed
- joint Jrl4_wheel: axis 1.000000000e+00 0.000000000e+00 0.000000000e+00 -> (none); limit lower=0.0 upper=0.0 effort=40.0 velocity=33.510321638291124 -> (none); type continuous -> fixed
- joint Jrr4_wheel: axis -1.000000000e+00 0.000000000e+00 0.000000000e+00 -> (none); limit lower=0.0 upper=0.0 effort=40.0 velocity=33.510321638291124 -> (none); type continuous -> fixed
