Commit message: 7.7

File: src/ToGo.Prototype/urdf/ToGo.Prototype_abs.urdf (robot description, URDF)
Before this commit: robot Xtellar.Robotics/ToGo.Prototype, 23 links, 22 joints
Links:
- link L0_body_front: geometry collision mesh filename=file:///home/mm/opendog_quadruped/src/ToGo.Prototype/meshes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 scale=1.000000000e-03 1.000000000e-03 1.000000000e-03; visual mesh filename=file:///home/mm/opendog_quadruped/src/ToGo.Prototype/meshes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 scale=1.000000000e-03 1.000000000e-03 1.000000000e-03
- link L1_body_rear: geometry collision mesh filename=file:///home/mm/opendog_quadruped/src/ToGo.Prototype/meshes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 scale=1.000000000e-03 1.000000000e-03 1.000000000e-03; visual mesh filename=file:///home/mm/opendog_quadruped/src/ToGo.Prototype/meshes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 scale=1.000000000e-03 1.000000000e-03 1.000000000e-03
- link Lfl1_hip_roll: geometry collision mesh filename=file:///home/mm/opendog_quadruped/src/ToGo.Prototype/meshes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 scale=1.000000000e-03 1.000000000e-03 1.000000000e-03; visual mesh filename=file:///home/mm/opendog_quadruped/src/ToGo.Prototype/meshes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 scale=1.000000000e-03 1.000000000e-03 1.000000000e-03
- link Lfl2_hip_pitch: geometry collision mesh filename=file:///home/mm/opendog_quadruped/src/ToGo.Prototype/meshes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 scale=1.000000000e-03 1.000000000e-03 1.000000000e-03; visual mesh filename=file:///home/mm/opendog_quadruped/src/ToGo.Prototype/meshes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 scale=1.000000000e-03 1.000000000e-03 1.000000000e-03
- link Lfl3_knee: geometry collision mesh filename=file:///home/mm/opendog_quadruped/src/ToGo.Prototype/meshes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 scale=1.000000000e-03 1.000000000e-03 1.000000000e-03; visual mesh filename=file:///home/mm/opendog_quadruped/src/ToGo.Prototype/meshes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 scale=1.000000000e-03 1.000000000e-03 1.000000000e-03
- link Lfl4_wheel: geometry collision mesh filename=file:///home/mm/opendog_quadruped/src/ToGo.Prototype/meshes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 scale=1.000000000e-03 1.000000000e-03 1.000000000e-03; visual mesh filename=file:///home/mm/opendog_quadruped/src/ToGo.Prototype/meshes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 scale=1.000000000e-03 1.000000000e-03 1.000000000e-03
- link Lfr1_hip_roll: geometry collision mesh filename=file:///home/mm/opendog_quadruped/src/ToGo.Prototype/meshes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 scale=1.000000000e-03 1.000000000e-03 1.000000000e-03; visual mesh filename=file:///home/mm/opendog_quadruped/src/ToGo.Prototype/meshes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 scale=1.000000000e-03 1.000000000e-03 1.000000000e-03
- link Lfr2_hip_pitch: geometry collision mesh filename=file:///home/mm/opendog_quadruped/src/ToGo.Prototype/meshes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 scale=1.000000000e-03 1.000000000e-03 1.000000000e-03; visual mesh filename=file:///home/mm/opendog_quadruped/src/ToGo.Prototype/meshes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 scale=1.000000000e-03 1.000000000e-03 1.000000000e-03
- link Lfr3_knee: geometry collision mesh filename=file:///home/mm/opendog_quadruped/src/ToGo.Prototype/meshes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 scale=1.000000000e-03 1.000000000e-03 1.000000000e-03; visual mesh filename=file:///home/mm/opendog_quadruped/src/ToGo.Prototype/meshes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 scale=1.000000000e-03 1.000000000e-03 1.000000000e-03
- link Lfr4_wheel: geometry collision mesh filename=file:///home/mm/opendog_quadruped/src/ToGo.Prototype/meshes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 scale=1.000000000e-03 1.000000000e-03 1.000000000e-03; visual mesh filename=file:///home/mm/opendog_quadruped/src/ToGo.Prototype/meshes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 scale=1.000000000e-03 1.000000000e-03 1.000000000e-03
- link Lrl1_hip_roll: geometry collision mesh filename=file:///home/mm/opendog_quadruped/src/ToGo.Prototype/meshes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 scale=1.000000000e-03 1.000000000e-03 1.000000000e-03; visual mesh filename=file:///home/mm/opendog_quadruped/src/ToGo.Prototype/meshes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 scale=1.000000000e-03 1.000000000e-03 1.000000000e-03
- link Lrl2_hip_pitch: geometry collision mesh filename=file:///home/mm/opendog_quadruped/src/ToGo.Prototype/meshes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 scale=1.000000000e-03 1.000000000e-03 1.000000000e-03; visual mesh filename=file:///home/mm/opendog_quadruped/src/ToGo.Prototype/meshes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 scale=1.000000000e-03 1.000000000e-03 1.000000000e-03
- link Lrl3_knee: geometry collision mesh filename=file:///home/mm/opendog_quadruped/src/ToGo.Prototype/meshes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 scale=1.000000000e-03 1.000000000e-03 1.000000000e-03; visual mesh filename=file:///home/mm/opendog_quadruped/src/ToGo.Prototype/meshes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 scale=1.000000000e-03 1.000000000e-03 1.000000000e-03
- link Lrl4_wheel: geometry collision mesh filename=file:///home/mm/opendog_quadruped/src/ToGo.Prototype/meshes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 scale=1.000000000e-03 1.000000000e-03 1.000000000e-03; visual mesh filename=file:///home/mm/opendog_quadruped/src/ToGo.Prototype/meshes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 scale=1.000000000e-03 1.000000000e-03 1.000000000e-03
- link Lrr1_hip_roll: geometry collision mesh filename=file:///home/mm/opendog_quadruped/src/ToGo.Prototype/meshes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 scale=1.000000000e-03 1.000000000e-03 1.000000000e-03; visual mesh filename=file:///home/mm/opendog_quadruped/src/ToGo.Prototype/meshes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 scale=1.000000000e-03 1.000000000e-03 1.000000000e-03
- link Lrr2_hip_pitch: geometry collision mesh filename=file:///home/mm/opendog_quadruped/src/ToGo.Prototype/meshes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 scale=1.000000000e-03 1.000000000e-03 1.000000000e-03; visual mesh filename=file:///home/mm/opendog_quadruped/src/ToGo.Prototype/meshes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 scale=1.000000000e-03 1.000000000e-03 1.000000000e-03
- link Lrr3_knee: geometry collision mesh filename=file:///home/mm/opendog_quadruped/src/ToGo.Prototype/meshes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 scale=1.000000000e-03 1.000000000e-03 1.000000000e-03; visual mesh filename=file:///home/mm/opendog_quadruped/src/ToGo.Prototype/meshes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 scale=1.000000000e-03 1.000000000e-03 1.000000000e-03
- link Lrr4_wheel: geometry collision mesh filename=file:///home/mm/opendog_quadruped/src/ToGo.Prototype/meshes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 scale=1.000000000e-03 1.000000000e-03 1.000000000e-03; visual mesh filename=file:///home/mm/opendog_quadruped/src/ToGo.Prototype/meshes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 scale=1.000000000e-03 1.000000000e-03 1.000000000e-03
